File: hardware/Geiger_Mod/Geiger.sch (EAGLE design)
At the start: 20 parts, among them Q1 KSP44, Q2 2N3904, X1 GM-tube

Commit message: layout changes
Parts:
- removed R1: 1K, SparkFun-Electromechanical:TRIMPOTPTH
- C3, C4: device rcl:CPOL-USE3.5-8 -> rcl:CPOL-USE2.5-7
- renumbered X1 to GM
Connections:
- removed net N$14: JP3.7, SG1.1
- removed net N$15: PWM.P$1, R1.CW, R1.WIPER
- new net N$3: JP3.6, SG1.1
- net N$1: now also JP3.7, PWM.P$1; no longer R1.CCW
Changed lines of the file:
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@@
 <grid distance="0.1" unitdist="inch" unit="inch" style="lines" multiple="1" display="no" altdistance="0.01" altunitdist="inch" altunit="inch"/>
 <layers>
-<layer number="1" name="Top" color="4" fill="1" visible="yes" active="no"/>
-<layer number="16" name="Bottom" color="1" fill="1" visible="yes" active="no"/>
-<layer number="17" name="Pads" color="2" fill="1" visible="yes" active="no"/>
-<layer number="18" name="Vias" color="2" fill="1" visible="yes" active="no"/>
-<layer number="19" name="Unrouted" color="6" fill="1" visible="yes" active="no"/>
-<layer number="20" name="Dimension" color="15" fill="1" visible="yes" active="no"/>
-<layer number="21" name="tPlace" color="7" fill="1" visible="yes" active="no"/>
-<layer number="22" name="bPlace" color="7" fill="1" visible="yes" active="no"/>
-<layer number="23" name="tOrigins" color="15" fill="1" visible="yes" active="no"/>
-<layer number="24" name="bOrigins" color="15" fill="1" visible="yes" active="no"/>
-<layer number="25" name="tNames" color="7" fill="1" visible="yes" active="no"/>
-<layer number="26" name="bNames" color="7" fill="1" visible="yes" active="no"/>
-<layer number="27" name="tValues" color="7" fill="1" visible="yes" active="no"/>
-<layer number="28" name="bValues" color="7" fill="1" visible="yes" active="no"/>
+<layer number="1" name="Top" color="4" fill="1" visible="no" active="no"/>
+<layer number="16" name="Bottom" color="1" fill="1" visible="no" active="no"/>
+<layer number="17" name="Pads" color="2" fill="1" visible="no" active="no"/>
+<layer number="18" name="Vias" color="2" fill="1" visible="no" active="no"/>
+<layer number="19" name="Unrouted" color="6" fill="1" visible="no" active="no"/>
+<layer number="20" name="Dimension" color="15" fill="1" visible="no" active="no"/>
+<layer number="21" name="tPlace" color="7" fill="1" visible="no" active="no"/>
+<layer number="22" name="bPlace" color="7" fill="1" visible="no" active="no"/>
+<layer number="23" name="tOrigins" color="15" fill="1" visible="no" active="no"/>
+<layer number="24" name="bOrigins" color="15" fill="1" visible="no" active="no"/>
+<layer number="25" name="tNames" color="7" fill="1" visible="no" active="no"/>
+<layer number="26" name="bNames" color="7" fill="1" visible="no" active="no"/>
+<layer number="27" name="tValues" color="7" fill="1" visible="no" active="no"/>
+<layer number="28" name="bValues" color="7" fill="1" visible="no" active="no"/>
 <layer number="29" name="tStop" color="7" fill="3" visible="no" active="no"/>
 <layer number="30" name="bStop" color="7" fill="6" visible="no" active="no"/>
@@
 <layer number="35" name="tGlue" color="7" fill="4" visible="no" active="no"/>
 <layer number="36" name="bGlue" color="7" fill="5" visible="no" active="no"/>
-<layer number="37" name="tTest" color="7" fill="1" visible="yes" active="no"/>
-<layer number="38" name="bTest" color="7" fill="1" visible="yes" active="no"/>
+<layer number="37" name="tTest" color="7" fill="1" visible="no" active="no"/>
+<layer number="38" name="bTest" color="7" fill="1" visible="no" active="no"/>
 <layer number="39" name="tKeepout" color="4" fill="11" visible="no" active="no"/>
 <layer number="40" name="bKeepout" color="1" fill="11" visible="no" active="no"/>
@@
 <layer number="44" name="Drills" color="7" fill="1" visible="no" active="no"/>
 <layer number="45" name="Holes" color="7" fill="1" visible="no" active="no"/>
-<layer number="46" name="Milling" color="3" fill="1" visible="yes" active="no"/>
-<layer number="47" name="Measures" color="7" fill="1" visible="yes" active="no"/>
-<layer number="48" name="Document" color="7" fill="1" visible="yes" active="no"/>
-<layer number="49" name="Reference" color="7" fill="1" visible="yes" active="no"/>
-<layer number="50" name="dxf" color="7" fill="1" visible="yes" active="no"/>
-<layer number="51" name="wire" color="7" fill="1" visible="yes" active="no"/>
-<layer number="52" name="bDocu" color="7" fill="1" visible="yes" active="no"/>
-<layer number="53" name="tGND_GNDA" color="7" fill="1" visible="yes" active="no"/>
-<layer number="54" name="bGND_GNDA" color="7" fill="1" visible="yes" active="no"/>
-<layer number="56" name="wert" color="7" fill="1" visible="yes" active="no"/>
+<layer number="46" name="Milling" color="3" fill="1" visible="no" active="no"/>
+<layer number="47" name="Measures" color="7" fill="1" visible="no" active="no"/>
+<layer number="48" name="Document" color="7" fill="1" visible="no" active="no"/>
+<layer number="49" name="Reference" color="7" fill="1" visible="no" active="no"/>
+<layer number="50" name="dxf" color="7" fill="1" visible="no" active="no"/>
+<layer number="51" name="wire" color="7" fill="1" visible="no" active="no"/>
+<layer number="52" name="bDocu" color="7" fill="1" visible="no" active="no"/>
+<layer number="53" name="tGND_GNDA" color="7" fill="1" visible="no" active="no"/>
+<layer number="54" name="bGND_GNDA" color="7" fill="1" visible="no" active="no"/>
+<layer number="56" name="wert" color="7" fill="1" visible="no" active="no"/>
 <layer number="91" name="Nets" color="2" fill="1" visible="yes" active="yes"/>
 <layer number="92" name="Busses" color="1" fill="1" visible="yes" active="yes"/>
@@
 <part name="GND6" library="SparkFun" deviceset="GND" device=""/>
 <part name="JP3" library="SparkFun-Connectors" deviceset="M08" device="1X08" value="1"/>
-<part name="R1" library="SparkFun-Electromechanical" deviceset="TRIMPOT" device="PTH" value="1K"/>
 <part name="R2" library="rcl" deviceset="R-US_" device="0207/10" value="1K"/>
 <part name="Q1" library="transistor-npn" deviceset="BC550*" device="" technology="B" value="KSP44"/>
@@
 <part name="Q2" library="transistor-small-signal" deviceset="2N3904" device=""/>
 <part name="C1" library="rcl" deviceset="C-US" device="150-054X183" value="10nF,1000V"/>
-<part name="C3" library="rcl" deviceset="CPOL-US" device="E3.5-8" value="100uf,6.3V"/>
-<part name="C4" library="rcl" deviceset="CPOL-US" device="E3.5-8" value="100uf,6.3V"/>
+<part name="C3" library="rcl" deviceset="CPOL-US" device="E2.5-7" value="100uf,6.3V"/>
+<part name="C4" library="rcl" deviceset="CPOL-US" device="E2.5-7" value="100uf,6.3V"/>
 <part name="R3" library="rcl" deviceset="R-US_" device="0207/10" value="100"/>
 <part name="R4" library="rcl" deviceset="R-US_" device="0207/10" value="100k"/>
@@
 <part name="GND2" library="SparkFun" deviceset="GND" device=""/>
 <part name="GND4" library="SparkFun" deviceset="GND" device=""/>
-<part name="X1" library="con-phoenix-350" deviceset="1751248" device="" value="GM-tube"/>
+<part name="GM" library="con-phoenix-350" deviceset="1751248" device="" value="GM-tube"/>
 <part name="SG1" library="SparkFun-Electromechanical" deviceset="BUZZER" device="NS"/>
 <part name="PWM" library="1AA_Stofer" deviceset="SOLDER_POINT" device="A"/>
@@
 <instance part="GND6" gate="1" x="198.12" y="134.62"/>
 <instance part="JP3" gate="G$1" x="205.74" y="154.94" rot="R180"/>
-<instance part="R1" gate="R?" x="68.58" y="157.48" rot="R180"/>
 <instance part="R2" gate="G$1" x="96.52" y="157.48" rot="R180"/>
 <instance part="Q1" gate="G$1" x="114.3" y="157.48"/>
@@
 <instance part="GND2" gate="1" x="96.52" y="175.26"/>
 <instance part="GND4" gate="1" x="147.32" y="177.8"/>
-<instance part="X1" gate="-1" x="160.02" y="170.18"/>
-<instance part="X1" gate="-2" x="160.02" y="165.1"/>
+<instance part="GM" gate="-1" x="160.02" y="170.18"/>
+<instance part="GM" gate="-2" x="160.02" y="165.1"/>
 <instance part="SG1" gate="G$1" x="182.88" y="147.32" rot="MR270"/>
 <instance part="PWM" gate="G$1" x="63.5" y="167.64" rot="R90"/>
@@
 <net name="N$1" class="0">
 <segment>
-<pinref part="R1" gate="R?" pin="CCW"/>
 <pinref part="R2" gate="G$1" pin="2"/>
-<wire x1="91.44" y1="157.48" x2="73.66" y2="157.48" width="0.1524" layer="91"/>
+<wire x1="91.44" y1="157.48" x2="88.9" y2="157.48" width="0.1524" layer="91"/>
+<pinref part="PWM" gate="G$1" pin="P$1"/>
+<wire x1="88.9" y1="157.48" x2="63.5" y2="157.48" width="0.1524" layer="91"/>
+<wire x1="88.9" y1="157.48" x2="88.9" y2="121.92" width="0.1524" layer="91"/>
+<wire x1="88.9" y1="121.92" x2="190.5" y2="121.92" width="0.1524" layer="91"/>
+<wire x1="190.5" y1="121.92" x2="190.5" y2="147.32" width="0.1524" layer="91"/>
+<pinref part="JP3" gate="G$1" pin="7"/>
+<wire x1="190.5" y1="147.32" x2="200.66" y2="147.32" width="0.1524" layer="91"/>
 </segment>
 </net>
@@
 <wire x1="142.24" y1="170.18" x2="142.24" y2="165.1" width="0.1524" layer="91"/>
 <wire x1="142.24" y1="170.18" x2="157.48" y2="170.18" width="0.1524" layer="91"/>
-<pinref part="X1" gate="-1" pin="K"/>
+<pinref part="GM" gate="-1" pin="K"/>
 </segment>
 </net>
@@
 <wire x1="154.94" y1="165.1" x2="147.32" y2="165.1" width="0.1524" layer="91"/>
 <wire x1="147.32" y1="165.1" x2="147.32" y2="152.4" width="0.1524" layer="91"/>
-<pinref part="X1" gate="-2" pin="K"/>
-</segment>
-</net>
-<net name="N$14" class="0">
+<pinref part="GM" gate="-2" pin="K"/>
+</segment>
+</net>
+<net name="N$3" class="0">
 <segment>
 <pinref part="SG1" gate="G$1" pin="1"/>
-<pinref part="JP3" gate="G$1" pin="7"/>
-<wire x1="185.42" y1="147.32" x2="200.66" y2="147.32" width="0.1524" layer="91"/>
-</segment>
-</net>
-<net name="N$15" class="0">
-<segment>
-<pinref part="R1" gate="R?" pin="CW"/>
-<pinref part="PWM" gate="G$1" pin="P$1"/>
-<pinref part="R1" gate="R?" pin="WIPER"/>
-<wire x1="68.58" y1="152.4" x2="63.5" y2="152.4" width="0.1524" layer="91"/>
-<wire x1="63.5" y1="152.4" x2="63.5" y2="157.48" width="0.1524" layer="91"/>
-</segment>
-</net>
+<wire x1="185.42" y1="147.32" x2="185.42" y2="149.86" width="0.1524" layer="91"/>
+<pinref part="JP3" gate="G$1" pin="6"/>
+<wire x1="185.42" y1="149.86" x2="200.66" y2="149.86" width="0.1524" layer="91"/>
+</segment>
+</net>
